File: swadge-c3/swadge-c3.kicad_pcb (KiCad board)
At the start: 2 copper layers, 73.7 x 89.4 mm, 68 parts, among them J1 USB_B_Micro, SW1 4-1437565-2, SW2 4-1437565-2, SW3 4-1437565-2, SW4 4-1437565-2, SW5 4-1437565-2, SW6 4-1437565-2, SW7 4-1437565-2, SW8 4-1437565-2, SW9 SW_SPDT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

Commit message: Replaced QMA6981 with QMA7981. Updated art. Updated renders
Parts:
- U7: value QMA6981 -> QMA7981
Connections:
- U4 pad A9: IO4_SW2 -> IO1_RES
- U4 pad B9: IO1_RES -> IO4_SW2
- U7 pad 10: Net-(U7-Pad10) -> +3V3
Routing:
- net +3V3: track 358.6 -> 361.2 mm
- net IO4_SW2: vias 3 -> 2
- net IO1_RES: vias 2 -> 3
- net GND: vias 42 -> 44
